File: hardware/fmcw2/fmcw2.kicad_pcb (KiCad board)
At the start: 4 copper layers, 40.3 x 22.9 mm, 136 parts, among them P1 CONN_15X2, Q1 SSM3K15AFS, U1 ADF4158, U10 HMC431LP4, U11 SKY65404, U12 PAT1220-6dB, U13 SMA, U14 MGA-25203, U15 SMA, U16 HMC313, U19 LDS3985, U2 SG-210STF 30MHz, U3 PAT1220-6dB, U4 5400BL15B050E, U5 LT6232, U6 ADL5801, U7 TLV271, U8 5400BL15B050E, U9 MCP1700

Commit message: Increase PLL loop bandwidth
Faster frequency settling
Parts:
- C10: value 330n -> 2.2n
- C14: value 10n -> 100p
- C29: value 470p -> 18p
- C42: value 1n -> 470p
- C55: value 2n -> 2.2n
- C56, C57: value 1u -> 330n
- L3: value 4.7n(L-07C4N7SV6T) -> LQW15AN9N9J80D
- R1: value 5.5k -> 5.49k
- R10: value 7k -> 6.98k
- R13: value 0 -> DNP
- R14: value 40k -> 39k
- R18: value 8.3k -> 8.25k
- R2: value 69.8 -> 750
- R21: value DNP -> 1k
- R23: value 550 -> 549
- R24, R25: value 100 -> 549
- R28, R29: value 550 -> 1k
- R32, R33: value 5k -> 4.99k
- R4: value 240 -> 2.2k
Changed lines of the file:
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@@
-(kicad_pcb (version 4) (host pcbnew "(2015-07-13 BZR 5934)-product")
+(kicad_pcb (version 4) (host pcbnew "(2015-12-18 BZR 6383)-product")
   (general
     (links 358)
@@
   )
   (setup
-    (last_trace_width 0.34)
+    (last_trace_width 0.15)
     (user_trace_width 0.2)
     (user_trace_width 0.34)
@@
       (effects (font (size 0.5 0.5) (thickness 0.125)))
     )
-    (fp_text value "4.7n(L-07C4N7SV6T)" (at 0 1.7 90) (layer F.Fab)
+    (fp_text value LQW15AN9N9J80D (at 0 1.7 90) (layer F.Fab)
       (effects (font (size 1 1) (thickness 0.15)))
     )
@@
       (effects (font (size 0.5 0.5) (thickness 0.125)))
     )
-    (fp_text value 330n (at 0 1.7 270) (layer F.Fab)
+    (fp_text value 2.2n (at 0 1.7 270) (layer F.Fab)
       (effects (font (size 1 1) (thickness 0.15)))
     )
@@
       (effects (font (size 0.5 0.5) (thickness 0.125)))
     )
-    (fp_text value 10n (at 0 1.7 270) (layer F.Fab)
+    (fp_text value 100p (at 0 1.7 270) (layer F.Fab)
       (effects (font (size 1 1) (thickness 0.15)))
     )
@@
       (effects (font (size 0.5 0.5) (thickness 0.125)) (justify mirror))
     )
-    (fp_text value 470p (at 0 -1.7 270) (layer B.Fab)
+    (fp_text value 18p (at 0 -1.7 270) (layer B.Fab)
       (effects (font (size 1 1) (thickness 0.15)) (justify mirror))
     )
@@
       (effects (font (size 0.5 0.5) (thickness 0.125)))
     )
-    (fp_text value 1n (at 0 1.7 180) (layer F.Fab)
+    (fp_text value 470p (at 0 1.7 180) (layer F.Fab)
       (effects (font (size 1 1) (thickness 0.15)))
     )
@@
       (effects (font (size 0.5 0.5) (thickness 0.125)) (justify mirror))
     )
-    (fp_text value 2n (at 0 -1.7 270) (layer B.Fab)
+    (fp_text value 2.2n (at 0 -1.7 270) (layer B.Fab)
       (effects (font (size 1 1) (thickness 0.15)) (justify mirror))
     )
@@
       (effects (font (size 0.5 0.5) (thickness 0.125)) (justify mirror))
     )
-    (fp_text value 1u (at 0 -1.9) (layer B.Fab)
+    (fp_text value 330n (at 0 -1.9) (layer B.Fab)
       (effects (font (size 1 1) (thickness 0.15)) (justify mirror))
     )
@@
       (effects (font (size 0.5 0.5) (thickness 0.125)) (justify mirror))
     )
-    (fp_text value 1u (at 0 -1.9) (layer B.Fab)
+    (fp_text value 330n (at 0 -1.9) (layer B.Fab)
       (effects (font (size 1 1) (thickness 0.15)) (justify mirror))
     )
@@
       (effects (font (size 0.5 0.5) (thickness 0.125)))
     )
-    (fp_text value 5.5k (at 0 1.8) (layer F.Fab)
+    (fp_text value 5.49k (at 0 1.8) (layer F.Fab)
       (effects (font (size 1 1) (thickness 0.15)))
     )
@@
       (effects (font (size 0.5 0.5) (thickness 0.125)) (justify mirror))
     )
-    (fp_text value 69.8 (at 0 -1.8 270) (layer B.Fab)
+    (fp_text value 750 (at 0 -1.8 270) (layer B.Fab)
       (effects (font (size 1 1) (thickness 0.15)) (justify mirror))
     )
@@
       (effects (font (size 0.5 0.5) (thickness 0.125)))
     )
-    (fp_text value 240 (at 0 1.8) (layer F.Fab)
+    (fp_text value 2.2k (at 0 1.8) (layer F.Fab)
       (effects (font (size 1 1) (thickness 0.15)))
     )
@@
       (effects (font (size 0.5 0.5) (thickness 0.125)) (justify mirror))
     )
-    (fp_text value 7k (at 0 -1.8 180) (layer B.Fab)
+    (fp_text value 6.98k (at 0 -1.8 180) (layer B.Fab)
       (effects (font (size 1 1) (thickness 0.15)) (justify mirror))
     )
@@
       (effects (font (size 0.5 0.5) (thickness 0.125)) (justify mirror))
     )
-    (fp_text value 0 (at 0 -1.8 180) (layer B.Fab)
+    (fp_text value DNP (at 0 -1.8 180) (layer B.Fab)
       (effects (font (size 1 1) (thickness 0.15)) (justify mirror))
     )
@@
       (effects (font (size 0.5 0.5) (thickness 0.125)) (justify mirror))
     )
-    (fp_text value 40k (at 0 -1.8) (layer B.Fab)
+    (fp_text value 39k (at 0 -1.8) (layer B.Fab)
       (effects (font (size 1 1) (thickness 0.15)) (justify mirror))
     )
@@
       (effects (font (size 0.5 0.5) (thickness 0.125)) (justify mirror))
     )
-    (fp_text value 8.3k (at 0 -1.8 180) (layer B.Fab)
+    (fp_text value 8.25k (at 0 -1.8 180) (layer B.Fab)
       (effects (font (size 1 1) (thickness 0.15)) (justify mirror))
     )
@@
       (effects (font (size 0.5 0.5) (thickness 0.125)) (justify mirror))
     )
-    (fp_text value DNP (at 0 -1.8) (layer B.Fab)
+    (fp_text value 1k (at 0 -1.8) (layer B.Fab)
       (effects (font (size 1 1) (thickness 0.15)) (justify mirror))
     )
@@
       (effects (font (size 0.5 0.5) (thickness 0.125)))
     )
-    (fp_text value 550 (at 0 1.8 90) (layer F.Fab)
+    (fp_text value 549 (at 0 1.8 90) (layer F.Fab)
       (effects (font (size 1 1) (thickness 0.15)))
     )
@@
       (effects (font (size 0.5 0.5) (thickness 0.125)) (justify mirror))
     )
-    (fp_text value 100 (at 0 -1.8) (layer B.Fab)
+    (fp_text value 549 (at 0 -1.8) (layer B.Fab)
       (effects (font (size 1 1) (thickness 0.15)) (justify mirror))
     )
@@
       (effects (font (size 0.5 0.5) (thickness 0.125)) (justify mirror))
     )
-    (fp_text value 100 (at 0 -1.8) (layer B.Fab)
+    (fp_text value 549 (at 0 -1.8) (layer B.Fab)
       (effects (font (size 1 1) (thickness 0.15)) (justify mirror))
     )
@@
       (effects (font (size 0.5 0.5) (thickness 0.125)) (justify mirror))
     )
-    (fp_text value 550 (at 0 -1.8 180) (layer B.Fab)
+    (fp_text value 1k (at 0 -1.8 180) (layer B.Fab)
       (effects (font (size 1 1) (thickness 0.15)) (justify mirror))
     )
@@
       (effects (font (size 0.5 0.5) (thickness 0.125)))
     )
-    (fp_text value 550 (at 0 1.8 180) (layer F.Fab)
+    (fp_text value 1k (at 0 1.8 180) (layer F.Fab)
       (effects (font (size 1 1) (thickness 0.15)))
     )
@@
       (effects (font (size 0.5 0.5) (thickness 0.125)) (justify mirror))
     )
-    (fp_text value 5k (at 0 -1.8 180) (layer B.Fab)
+    (fp_text value 4.99k (at 0 -1.8 180) (layer B.Fab)
       (effects (font (size 1 1) (thickness 0.15)) (justify mirror))
     )
@@
       (effects (font (size 0.5 0.5) (thickness 0.125)) (justify mirror))
     )
-    (fp_text value 5k (at 0 -1.8 180) (layer B.Fab)
+    (fp_text value 4.99k (at 0 -1.8 180) (layer B.Fab)
       (effects (font (size 1 1) (thickness 0.15)) (justify mirror))
     )
